File: EAGLE/virtual_wall_lp.sch (EAGLE design)
At the start: 29 parts, among them U1 PIC12F683-I/SN, U2 CAT3200TDI-GT3, U3 BSS138-7-F, Y1 CRYSTAL.ABS07

Commit message: added missing net from charge pump to ucontroller vdd
Connections:
- removed net N$16: C4.1, U1.VDD
- net VDD: now also C4.1, U1.VDD
Changed lines of the file:
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@@
 <label x="-53.34" y="53.34" size="1.778" layer="95"/>
+</segment>
+<segment>
+<pinref part="U1" gate="A" pin="VDD"/>
+<wire x1="-241.3" y1="38.1" x2="-246.38" y2="38.1" width="0.1524" layer="91"/>
+<pinref part="C4" gate="G$1" pin="1"/>
+<wire x1="-246.38" y1="35.56" x2="-246.38" y2="38.1" width="0.1524" layer="91"/>
+<label x="-248.92" y="38.1" size="1.778" layer="95"/>
 </segment>
 </net>
@@
 </segment>
 </net>
-<net name="N$16" class="1">
-<segment>
-<pinref part="U1" gate="A" pin="VDD"/>
-<wire x1="-241.3" y1="38.1" x2="-246.38" y2="38.1" width="0.1524" layer="91"/>
-<pinref part="C4" gate="G$1" pin="1"/>
-<wire x1="-246.38" y1="35.56" x2="-246.38" y2="38.1" width="0.1524" layer="91"/>
-</segment>
-</net>
